Commit message: format dummy urdf

File: res/robot/dummy_robot/urdf/dummy_ros_sim.urdf (robot description, URDF)
Before this commit: robot dummy_ros_sim, 7 links, 6 joints
Links:
- link base_link: geometry collision mesh filename=meshes/base_link.STL; visual mesh filename=meshes/base_link.STL
- link link1: geometry collision mesh filename=meshes/link1.STL; visual mesh filename=meshes/link1.STL
- link link2: geometry collision mesh filename=meshes/link2.STL; visual mesh filename=meshes/link2.STL
- link link3: geometry collision mesh filename=meshes/link3.STL; visual mesh filename=meshes/link3.STL
- link link4: geometry collision mesh filename=meshes/link4.STL; visual mesh filename=meshes/link4.STL
- link link5: geometry collision mesh filename=meshes/link5.STL; visual mesh filename=meshes/link5.STL
- link link6: geometry collision mesh filename=meshes/link6.STL; visual mesh filename=meshes/link6.STL
Joints:
- joint joint2: origin xyz=-0.035 -0.021695 0.02275 rpy=1.5708 0 0 -> xyz=-0.035 -0.021695 0.02275 rpy=-1.5708 0 0

Commit message: fixed bug RPY order Z-Y-X

File: res/robot/dummy_robot/urdf/dummy_ros_sim.urdf (robot description, URDF)
Before this commit: robot dummy_ros_sim, 7 links, 6 joints
Joints:
- joint joint2: origin xyz=-0.035 -0.021695 0.02275 rpy=-1.5708 0 0 -> xyz=-0.035 -0.021695 0.02275 rpy=1.5708 0 0
